Commit message: edit the code and make it shorter

File: urdf/lidar.xacro (robot description, xacro)
@@ -2,5 +2,5 @@
 <robot xmlns:xacro="http://www.ros.org/wiki/xacro" >
     <joint name="chassis_to_lidar" type="fixed">
-        <origin xyz="0.0 0.0 0.22" rpy="0.0 0.0 0"/>
+        <origin xyz="0.5 0.0 0.22" rpy="0.0 0.0 0"/>
         <parent link="chassis"/>
         <child link="hokuyo_link"/>
